Commit message: Fixing the wrong path to the model files in the URDF

File: robot_model/mpo_700/mpo_700.urdf (robot description, URDF)
Before this commit: robot mpo_700, 12 links, 11 joints
Links:
- link base_footprint: geometry collision mesh filename=package://neo_mpo_700-2/robot_model/mpo_700/meshes/MPO-700-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 scale=0.001 0.001 0.001; visual mesh filename=package://neo_mpo_700-2/robot_model/mpo_700/meshes/MPO-700-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 scale=0.001 0.001 0.001
- link lidar_1_link: geometry collision mesh filename=package://neo_mpo_700-2/robot_model/mpo_700/meshes/SICK-S30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 scale=0.001 0.001 0.001; visual mesh filename=package://neo_mpo_700-2/robot_model/mpo_700/meshes/SICK-S30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 scale=0.001 0.001 0.001
- link lidar_2_link: geometry collision mesh filename=package://neo_mpo_700-2/robot_model/mpo_700/meshes/SICK-S30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 scale=0.001 0.001 0.001; visual mesh filename=package://neo_mpo_700-2/robot_model/mpo_700/meshes/SICK-S30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 scale=0.001 0.001 0.001
- link mpo_700_caster_back_left_link: geometry collision mesh filename=package://neo_mpo_700-2/robot_model/mpo_700/meshes/MPO-700-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 scale=0.001 0.001 0.001; visual mesh filename=package://neo_mpo_700-2/robot_model/mpo_700/meshes/MPO-700-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 scale=0.001 0.001 0.001
- link mpo_700_caster_back_right_link: geometry collision mesh filename=package://neo_mpo_700-2/robot_model/mpo_700/meshes/MPO-700-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 scale=0.001 0.001 0.001; visual mesh filename=package://neo_mpo_700-2/robot_model/mpo_700/meshes/MPO-700-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 scale=0.001 0.001 0.001
- link mpo_700_caster_front_left_link: geometry collision mesh filename=package://neo_mpo_700-2/robot_model/mpo_700/meshes/MPO-700-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 scale=0.001 0.001 0.001; visual mesh filename=package://neo_mpo_700-2/robot_model/mpo_700/meshes/MPO-700-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 scale=0.001 0.001 0.001
- link mpo_700_caster_front_right_link: geometry collision mesh filename=package://neo_mpo_700-2/robot_model/mpo_700/meshes/MPO-700-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 scale=0.001 0.001 0.001; visual mesh filename=package://neo_mpo_700-2/robot_model/mpo_700/meshes/MPO-700-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 scale=0.001 0.001 0.001
- link mpo_700_wheel_back_left_link: geometry collision mesh filename=package://neo_mpo_700-2/robot_model/mpo_700/meshes/MPO-700-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 scale=0.001 0.001 0.001; visual mesh filename=package://neo_mpo_700-2/robot_model/mpo_700/meshes/MPO-700-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 scale=0.001 0.001 0.001
- link mpo_700_wheel_back_right_link: geometry collision mesh filename=package://neo_mpo_700-2/robot_model/mpo_700/meshes/MPO-700-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 scale=0.001 0.001 0.001; visual mesh filename=package://neo_mpo_700-2/robot_model/mpo_700/meshes/MPO-700-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 scale=0.001 0.001 0.001
- link mpo_700_wheel_front_left_link: geometry collision mesh filename=package://neo_mpo_700-2/robot_model/mpo_700/meshes/MPO-700-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 scale=0.001 0.001 0.001; visual mesh filename=package://neo_mpo_700-2/robot_model/mpo_700/meshes/MPO-700-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 scale=0.001 0.001 0.001
- link mpo_700_wheel_front_right_link: geometry collision mesh filename=package://neo_mpo_700-2/robot_model/mpo_700/meshes/MPO-700-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 scale=0.001 0.001 0.001; visual mesh filename=package://neo_mpo_700-2/robot_model/mpo_700/meshes/MPO-700-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 scale=0.001 0.001 0.001

Commit message: updating the robot model to visualize the joint states in RViz

File: robot_model/mpo_700/mpo_700.urdf (robot description, URDF)
Before this commit: robot mpo_700, 12 links, 11 joints
Links:
- link base_footprint: mass 30 -> 140
- link mpo_700_caster_back_left_link: mass 9 -> 12.7
- link mpo_700_caster_back_right_link: mass 9 -> 12.7
- link mpo_700_caster_front_left_link: mass 9 -> 12.7
- link mpo_700_caster_front_right_link: mass 9 -> 12.7
- link mpo_700_wheel_back_left_link: mass 2 -> 1.2; geometry collision sphere radius=0.09; visual mesh filename=package://neo_mpo_700-2/robot_model/mpo_700/meshes/MPO-700-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 scale=0.001 0.001 0.001
- link mpo_700_wheel_back_right_link: mass 2 -> 1.2; geometry collision sphere radius=0.09; visual mesh filename=package://neo_mpo_700-2/robot_model/mpo_700/meshes/MPO-700-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 scale=0.001 0.001 0.001
- link mpo_700_wheel_front_left_link: mass 2 -> 1.2; geometry collision sphere radius=0.09; visual mesh filename=package://neo_mpo_700-2/robot_model/mpo_700/meshes/MPO-700-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 scale=0.001 0.001 0.001
- link mpo_700_wheel_front_right_link: mass 2 -> 1.2; geometry collision sphere radius=0.09; visual mesh filename=package://neo_mpo_700-2/robot_model/mpo_700/meshes/MPO-700-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 scale=0.001 0.001 0.001
Joints:
- joint mpo_700_caster_back_left_joint: axis 0 0 -1 -> 0 0 1; limit (none) -> lower=-1e+16 upper=1e+16 effort=1000.0 velocity=6.5; origin xyz=0.24 -0.18 0.27 rpy=3.14 0 1.57 -> xyz=-0.24 0.18 0.22 rpy=0 0 3.14; type fixed -> revolute
- joint mpo_700_caster_back_right_joint: axis 0 0 -1 -> 0 0 1; limit (none) -> lower=-1e+16 upper=1e+16 effort=1000.0 velocity=6.5; origin xyz=-0.24 0.18 0.27 rpy=3.14 0 -1.57 -> xyz=-0.24 -0.18 0.22 rpy=0 0 0; type fixed -> revolute
- joint mpo_700_caster_front_left_joint: axis 0 0 -1 -> 0 0 1; limit (none) -> lower=-1e+16 upper=1e+16 effort=1000.0 velocity=6.5; origin xyz=0.24 0.18 0.27 rpy=3.14 0 -1.57 -> xyz=0.24 0.18 0.22 rpy=0 0 3.14; type fixed -> revolute
- joint mpo_700_caster_front_right_joint: axis 0 0 -1 -> 0 0 1; limit (none) -> lower=-1e+16 upper=1e+16 effort=1000.0 velocity=6.5; origin xyz=-0.24 -0.18 0.27 rpy=3.14 0 1.57 -> xyz=0.24 -0.18 0.22 rpy=0 0 0; type fixed -> revolute
- joint mpo_700_wheel_back_left_joint: axis 1 0 0 -> 0 -1 0; limit lower=-1e+16 upper=1e+16 effort=1000.0 velocity=3.5 -> lower=-1e+16 upper=1e+16 effort=1000.0 velocity=20.5; origin xyz=-0.05 0. 0.18 rpy=0 0 0 -> xyz=0.0 0.045 -0.12 rpy=0 0 0; type fixed -> revolute
- joint mpo_700_wheel_back_right_joint: axis 1 0 0 -> 0 -1 0; limit lower=-1e+16 upper=1e+16 effort=1000.0 velocity=3.5 -> lower=-1e+16 upper=1e+16 effort=1000.0 velocity=20.5; origin xyz=-0.05 0. 0.18 rpy=0 0 0 -> xyz=0.0 -0.045 -0.12 rpy=0 0 3.14; type fixed -> revolute
- joint mpo_700_wheel_front_left_joint: axis 1 0 0 -> 0 -1 0; limit lower=-1e+16 upper=1e+16 effort=1000.0 velocity=3.5 -> lower=-1e+16 upper=1e+16 effort=1000.0 velocity=20.5; origin xyz=-0.05 0. 0.18 rpy=0 0 0 -> xyz=0.0 0.045 -0.12 rpy=0 0 0; type fixed -> revolute
- joint mpo_700_wheel_front_right_joint: axis 1 0 0 -> 0 -1 0; limit lower=-1e+16 upper=1e+16 effort=1000.0 velocity=3.5 -> lower=-1e+16 upper=1e+16 effort=1000.0 velocity=20.5; origin xyz=-0.05 0. 0.18 rpy=0 0 0 -> xyz=0.0 -0.045 -0.12 rpy=0 0 3.14; type fixed -> revolute

Commit message: adding the linear axis

File: robot_model/mpo_700/mpo_700.urdf (robot description, URDF)
Before this commit: robot mpo_700, 12 links, 11 joints
Links:
- added link linear_axis_fixed_link; collision mesh filename=package://neo_mpo_700-2/robot_model/mpo_700/meshes/linear_a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 scale=0.1 0.1 0.1; visual mesh filename=package://neo_mpo_700-2/robot_model/mpo_700/meshes/linear_a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 scale=0.1 0.1 0.1
- added link linear_axis_slide_link; collision mesh filename=package://neo_mpo_700-2/robot_model/mpo_700/meshes/linear_a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 scale=0.1 0.1 0.1; visual mesh filename=package://neo_mpo_700-2/robot_model/mpo_700/meshes/linear_a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 scale=0.1 0.1 0.1
Joints:
- added joint linear_axis_fixed_joint: type fixed, parent base_link, child linear_axis_fixed_link, origin xyz=0.0 0 0.35 rpy=0 0 1.57, axis 0 1 0
- added joint linear_axis_slide_joint: type prismatic, parent linear_axis_fixed_link, child linear_axis_slide_link, origin xyz=0.0 -0.314 0.0 rpy=0 0 -1.57, axis 0 0 1, limit lower=0.1 upper=0.7 effort=54.0 velocity=0.2

Commit message: tunings

File: robot_model/mpo_700/mpo_700.urdf (robot description, URDF)
Before this commit: robot mpo_700, 14 links, 13 joints
Joints:
- joint linear_axis_slide_joint: limit lower=0.1 upper=0.7 effort=54.0 velocity=0.2 -> lower=0.0 upper=0.68 effort=54.0 velocity=0.15
