Commit message: adding urdf.xacro and removing unwanted URDF and dae

File: robot_model/mpo_700/mpo_700.urdf.xacro (robot description, xacro)
@@ -1,13 +1,22 @@
 <?xml version="1.0" ?>
-<!-- =================================================================================== -->
-<!-- |    This document was autogenerated by xacro from mpo_700.urdf.xacro             | -->
-<!-- |    EDITING THIS FILE BY HAND IS NOT RECOMMENDED                                 | -->
-<!-- =================================================================================== -->
-<robot name="mpo_700">
+<robot xmlns:xacro="http://www.ros.org/wiki/xacro" name="mpo_700">
   <!-- SENSORS -->
-  <!-- Sick S300 - Comment/Uncomment if required -->
-  <!-- Microscan - Comment/Uncomment if required -->
+  <xacro:arg name="arm_type" default=""/>
+  <xacro:arg name="use_imu" default="false"/>
+  <xacro:arg name="use_d435" default="false"/>
+  <xacro:property name="arm" value="$(arg arm_type)"/>
+  <xacro:property name="imu" value="$(arg use_imu)"/>
+  <xacro:property name="d435" value="$(arg use_d435)"/>
+  <!-- When there is an arm mounted, the joints of the wheels needs
+  to be of fixed type. The reason being, both the drive modules and
+  the arm cannot publish joint states simultenously. Thus we omit
+  the visualization of the drives. Issue will be fixed, when we switch
+  to ROS 2 control. -->
+  <xacro:property name="ODM_joint_type" value="revolute"/>
+  <xacro:unless value="${arm == ''}">
+    <xacro:property name="ODM_joint_type" value="fixed"/>
+  </xacro:unless>
   <link name="base_link"/>
-  <joint name="base_footprint_joint" type="fixed">
+  <joint name="base_footprint_joint" type="${ODM_joint_type}">
     <origin rpy="0 0 0" xyz="0 0 0"/>
     <axis xyz="0 0 -1"/>
@@ -36,6 +45,6 @@
     </collision>
   </link>
-  <joint name="mpo_700_caster_front_left_joint" type="revolute">
-    <origin rpy="0 0 3.14" xyz="0.24 0.18 0.22"/>
+  <joint name="mpo_700_caster_front_left_joint" type="${ODM_joint_type}">
+    <origin rpy="0 0 0" xyz="0.24 0.18 0.22"/>
     <axis xyz="0 0 1"/>
     <limit effort="1000.0" lower="-1e+16" upper="1e+16" velocity="6.5"/>
@@ -63,5 +72,5 @@
     </collision>
   </link>
-  <joint name="mpo_700_caster_front_right_joint" type="revolute">
+  <joint name="mpo_700_caster_front_right_joint" type="${ODM_joint_type}">
     <origin rpy="0 0 0" xyz="0.24 -0.18 0.22"/>
     <axis xyz="0 0 1"/>
@@ -90,6 +99,6 @@
     </collision>
   </link>
-  <joint name="mpo_700_caster_back_left_joint" type="revolute">
-    <origin rpy="0 0 3.14" xyz="-0.24 0.18 0.22"/>
+  <joint name="mpo_700_caster_back_left_joint" type="${ODM_joint_type}">
+    <origin rpy="0 0 0" xyz="-0.24 0.18 0.22"/>
     <axis xyz="0 0 1"/>
     <limit effort="1000.0" lower="-1e+16" upper="1e+16" velocity="6.5"/>
@@ -117,5 +126,5 @@
     </collision>
   </link>
-  <joint name="mpo_700_caster_back_right_joint" type="revolute">
+  <joint name="mpo_700_caster_back_right_joint" type="${ODM_joint_type}">
     <origin rpy="0 0 0" xyz="-0.24 -0.18 0.22"/>
     <axis xyz="0 0 1"/>
@@ -144,5 +153,5 @@
     </collision>
   </link>
-  <joint name="mpo_700_wheel_front_left_joint" type="revolute">
+  <joint name="mpo_700_wheel_front_left_joint" type="${ODM_joint_type}">
     <origin rpy="0 0 0" xyz="0.0 0.045 -0.12"/>
     <limit effort="1000.0" lower="-1e+16" upper="1e+16" velocity="20.5"/>
@@ -172,5 +181,5 @@
     </collision>
   </link>
-  <joint name="mpo_700_wheel_front_right_joint" type="revolute">
+  <joint name="mpo_700_wheel_front_right_joint" type="${ODM_joint_type}">
     <origin rpy="0 0 3.14" xyz="0.0 -0.045 -0.12"/>
     <limit effort="1000.0" lower="-1e+16" upper="1e+16" velocity="20.5"/>
@@ -200,5 +209,5 @@
     </collision>
   </link>
-  <joint name="mpo_700_wheel_back_left_joint" type="revolute">
+  <joint name="mpo_700_wheel_back_left_joint" type="${ODM_joint_type}">
     <origin rpy="0 0 0" xyz="0.0 0.045 -0.12"/>
     <limit effort="1000.0" lower="-1e+16" upper="1e+16" velocity="20.5"/>
@@ -228,5 +237,5 @@
     </collision>
   </link>
-  <joint name="mpo_700_wheel_back_right_joint" type="revolute">
+  <joint name="mpo_700_wheel_back_right_joint" type="${ODM_joint_type}">
     <origin rpy="0 0 3.14" xyz="0.0 -0.045 -0.12"/>
     <limit effort="1000.0" lower="-1e+16" upper="1e+16" velocity="20.5"/>
@@ -307,6 +316,14 @@
     </collision>
   </link>
-  <!-- uncomment if necessary -->
-  <!-- <link name="imu_link">
+  <!-- Realsense D435 -->
+  <xacro:if value="${d435 == True}">
+    <xacro:include filename="$(find realsense2_description)/urdf/_d435.urdf.xacro"/>
+    <xacro:sensor_d435 parent="base_link">
+      <origin xyz="0.292 0.0 0.716" rpy="0 0 0"/>
+    </xacro:sensor_d435>
+  </xacro:if>
+  <!-- Using IMU -->
+  <xacro:if value="${imu == True}">
+    <link name="imu_link">
       <inertial>
         <mass value="0.001" />
@@ -314,10 +331,65 @@
         <inertia ixx="0.0001" ixy="0" ixz="0" iyy="0.000001" iyz="0" izz="0.0001" />
       </inertial>
-  </link>
-  <joint name="imu2_joint" type="fixed">
-    <axis xyz="0 1 0"/>
-    <origin rpy="0 0 0" xyz="-0.052 0.208 0.266"/>
-    <parent link="base_link"/>
-    <child link="imu_link"/>
-  </joint> -->
+    </link>
+    <joint name="imu2_joint" type="fixed">
+      <axis xyz="0 1 0"/>
+      <origin rpy="0 0 0" xyz="-0.052 0.208 0.266"/>
+      <parent link="base_link"/>
+      <child link="imu_link"/>
+    </joint>
+  </xacro:if>
+  <xacro:unless value="${arm == ''}">
+    <xacro:arg name="tf_prefix" default="$(arg arm_type)" />
+    <xacro:arg name="joint_limit_params" default="$(find ur_description)/config/$(arg arm_type)/joint_limits.yaml"/>
+    <xacro:arg name="kinematics_params" default="$(find ur_description)/config/$(arg arm_type)/default_kinematics.yaml"/>
+    <xacro:arg name="physical_params" default="$(find ur_description)/config/$(arg arm_type)/physical_parameters.yaml"/>
+    <xacro:arg name="visual_params" default="$(find ur_description)/config/$(arg arm_type)/visual_parameters.yaml"/>
+    <xacro:arg name="transmission_hw_interface" default=""/>
+    <xacro:arg name="safety_limits" default="false"/>
+    <xacro:arg name="safety_pos_margin" default="0.15"/>
+    <xacro:arg name="safety_k_position" default="20"/>
+    <xacro:arg name="force_abs_paths" default="false" />
+    <!-- cabinet link -->
+    <joint name="cabinet_joint" type="fixed">
+      <origin rpy="0 0 0" xyz="0.025 0 0.35"/>
+      <joint_properties damping="1" friction="1"/>
+      <parent link="base_link"/>
+      <child link="cabinet_link"/>
+    </joint>
+    <link name="cabinet_link">
+    <inertial>
+      <mass value="2"/>
+      <origin rpy="0 0 0" xyz="0 0 0"/>
+      <inertia ixx="0.457072" ixy="0.0" ixz="0.0" iyy="0.23616" iyz="0.0" izz="0.686"/>
+    </inertial>
+    <visual>
+      <origin rpy="0 0 -1.5708" xyz="0 0 0"/>
+      <geometry>
+        <mesh filename="package://neo_mpo_700-2/robot_model/mpo_700/meshes/cabin.dae" scale="0.001 0.001 0.001"/>
+      </geometry>
+    </visual>
+    <collision>
+      <origin rpy="0 0 0" xyz="0. 0. 0"/>
+      <geometry>
+        <mesh filename="package://neo_mpo_700-2/robot_model/mpo_700/meshes/cabin.dae" scale="0.001 0.001 0.001"/>
+      </geometry>
+    </collision>
+    </link>
+    <!-- arm link -->
+    <xacro:include filename="$(find ur_description)/urdf/ur_macro.xacro"/>
+    <xacro:ur_robot name="$(arg arm_type)"
+      parent="cabinet_link"
+      tf_prefix="$(arg tf_prefix)"
+      joint_limits_parameters_file="$(arg joint_limit_params)"
+      kinematics_parameters_file="$(arg kinematics_params)"
+      physical_parameters_file="$(arg physical_params)"
+      visual_parameters_file="$(arg visual_params)"
+      safety_limits="$(arg safety_limits)"
+      safety_pos_margin="$(arg safety_pos_margin)"
+      safety_k_position="$(arg safety_k_position)"
+      >
+      <!-- position robot in the world -->
+      <origin xyz="0.133 0.0 0.416" rpy="0.0 0.0 0.0" />
+    </xacro:ur_robot>
+  </xacro:unless>
 </robot>

Commit message: adding opaque function to customize the launch

File: robot_model/mpo_700/mpo_700.urdf.xacro (robot description, xacro)
@@ -18,5 +18,5 @@
   </xacro:unless>
   <link name="base_link"/>
-  <joint name="base_footprint_joint" type="${ODM_joint_type}">
+  <joint name="base_footprint_joint" type="fixed">
     <origin rpy="0 0 0" xyz="0 0 0"/>
     <axis xyz="0 0 -1"/>

Commit message: adjusting the robot model

File: robot_model/mpo_700/mpo_700.urdf.xacro (robot description, xacro)
@@ -360,5 +360,5 @@
     <inertial>
       <mass value="2"/>
-      <origin rpy="0 0 0" xyz="0 0 0"/>
+      <origin rpy="0 0 -1.5708" xyz="0 0 0"/>
       <inertia ixx="0.457072" ixy="0.0" ixz="0.0" iyy="0.23616" iyz="0.0" izz="0.686"/>
     </inertial>
@@ -370,5 +370,5 @@
     </visual>
     <collision>
-      <origin rpy="0 0 0" xyz="0. 0. 0"/>
+      <origin rpy="0 0 -1.5708" xyz="0. 0. 0"/>
       <geometry>
         <mesh filename="package://neo_mpo_700-2/robot_model/mpo_700/meshes/cabin.dae" scale="0.001 0.001 0.001"/>
@@ -390,5 +390,5 @@
       >
       <!-- position robot in the world -->
-      <origin xyz="0.133 0.0 0.416" rpy="0.0 0.0 0.0" />
+      <origin xyz="0.133 0.0 0.416" rpy="0.0 0.0 -1.5708" />
     </xacro:ur_robot>
   </xacro:unless>

Commit message: adding gripper to the URDF and dependency update

File: robot_model/mpo_700/mpo_700.urdf.xacro (robot description, xacro)
@@ -5,7 +5,9 @@
   <xacro:arg name="use_imu" default="false"/>
   <xacro:arg name="use_d435" default="false"/>
+  <xacro:arg name="gripper_type" default=""/>
   <xacro:property name="arm" value="$(arg arm_type)"/>
   <xacro:property name="imu" value="$(arg use_imu)"/>
   <xacro:property name="d435" value="$(arg use_d435)"/>
+  <xacro:property name="gripper" value="$(arg gripper_type)"/>
   <!-- When there is an arm mounted, the joints of the wheels needs
   to be of fixed type. The reason being, both the drive modules and
@@ -392,4 +394,19 @@
       <origin xyz="0.133 0.0 0.416" rpy="0.0 0.0 -1.5708" />
     </xacro:ur_robot>
+    <xacro:unless value="${gripper == ''}">
+      <!-- ur_adapter for gripper-->
+      <xacro:include filename="$(find robotiq_description)/urdf/ur_to_robotiq_adapter.urdf.xacro"/>
+      <xacro:ur_to_robotiq
+          prefix=""
+          parent="$(arg tf_prefix)tool0"
+          child="neo_gripper_mount_link"
+          rotation="${pi/2}"
+          />
+      <!-- add gripper-->
+      <xacro:include filename="$(find robotiq_description)/urdf/robotiq_2f_140_macro.urdf.xacro"/>
+      <xacro:robotiq_gripper name="robotiq_gripper" prefix="" parent="neo_gripper_mount_link" include_ros2_control="true">
+          <origin xyz="0 0 0" rpy="0 0 -${pi / 2}"/>
+      </xacro:robotiq_gripper>
+    </xacro:unless>
   </xacro:unless>
 </robot>

Commit message: updates for fake hardware for gripper

File: robot_model/mpo_700/mpo_700.urdf.xacro (robot description, xacro)
@@ -6,8 +6,10 @@
   <xacro:arg name="use_d435" default="false"/>
   <xacro:arg name="gripper_type" default=""/>
+  <xacro:arg name="use_fake_hardware" default="false"/>
   <xacro:property name="arm" value="$(arg arm_type)"/>
   <xacro:property name="imu" value="$(arg use_imu)"/>
   <xacro:property name="d435" value="$(arg use_d435)"/>
   <xacro:property name="gripper" value="$(arg gripper_type)"/>
+  <xacro:property name="use_fake" value="$(arg use_fake_hardware)"/>
   <!-- When there is an arm mounted, the joints of the wheels needs
   to be of fixed type. The reason being, both the drive modules and
@@ -405,5 +407,9 @@
       <!-- add gripper-->
       <xacro:include filename="$(find robotiq_description)/urdf/robotiq_2f_140_macro.urdf.xacro"/>
-      <xacro:robotiq_gripper name="robotiq_gripper" prefix="" parent="neo_gripper_mount_link" include_ros2_control="true">
+      <xacro:robotiq_gripper name="robotiq_gripper"
+        prefix=""
+        parent="neo_gripper_mount_link"
+        include_ros2_control="true"
+        use_fake_hardware="${use_fake}">
           <origin xyz="0 0 0" rpy="0 0 -${pi / 2}"/>
       </xacro:robotiq_gripper>

Commit message: adding Epick gripper

File: robot_model/mpo_700/mpo_700.urdf.xacro (robot description, xacro)
@@ -5,5 +5,5 @@
   <xacro:arg name="use_imu" default="false"/>
   <xacro:arg name="use_d435" default="false"/>
-  <xacro:arg name="gripper_type" default=""/>
+  <xacro:arg name="gripper_type" default="2f_140"/>
   <xacro:arg name="use_fake_hardware" default="false"/>
   <xacro:property name="arm" value="$(arg arm_type)"/>
@@ -396,22 +396,32 @@
       <origin xyz="0.133 0.0 0.416" rpy="0.0 0.0 -1.5708" />
     </xacro:ur_robot>
+    <!-- add gripper-->
     <xacro:unless value="${gripper == ''}">
       <!-- ur_adapter for gripper-->
-      <xacro:include filename="$(find robotiq_description)/urdf/ur_to_robotiq_adapter.urdf.xacro"/>
-      <xacro:ur_to_robotiq
+      <xacro:if value="${gripper == '2f_140'}">
+        <xacro:include filename="$(find robotiq_description)/urdf/ur_to_robotiq_adapter.urdf.xacro"/>
+        <xacro:ur_to_robotiq
+            prefix=""
+            parent="$(arg tf_prefix)tool0"
+            child="neo_gripper_mount_link"
+            rotation="${pi/2}"
+            />
+        <xacro:include filename="$(find robotiq_description)/urdf/robotiq_2f_140_macro.urdf.xacro"/>
+        <xacro:robotiq_gripper name="robotiq_gripper"
           prefix=""
-          parent="$(arg tf_prefix)tool0"
-          child="neo_gripper_mount_link"
-          rotation="${pi/2}"
-          />
-      <!-- add gripper-->
-      <xacro:include filename="$(find robotiq_description)/urdf/robotiq_2f_140_macro.urdf.xacro"/>
-      <xacro:robotiq_gripper name="robotiq_gripper"
-        prefix=""
-        parent="neo_gripper_mount_link"
-        include_ros2_control="true"
-        use_fake_hardware="${use_fake}">
-          <origin xyz="0 0 0" rpy="0 0 -${pi / 2}"/>
-      </xacro:robotiq_gripper>
+          parent="neo_gripper_mount_link"
+          include_ros2_control="true"
+          use_fake_hardware="${use_fake}">
+            <origin xyz="0 0 0" rpy="0 0 -${pi / 2}"/>
+        </xacro:robotiq_gripper>
+      </xacro:if>
+      <xacro:if value="${gripper == 'epick'}">
+        <xacro:include filename="$(find epick_description)/urdf/epick_single_suction_cup.xacro"/>
+          <xacro:epick_single_suction_cup parent="$(arg tf_prefix)tool0"
+            use_fake_hardware="${use_fake}"
+            origin_xyz="0 0 0"
+            origin_rpy="0 0 -${pi / 2}"
+            />
+      </xacro:if>
     </xacro:unless>
   </xacro:unless>

Commit message: Feature/robotiq 2f 140 gripper and Epick (#49)
* Added Robotiq 2f 140 gripper to robot arm

* adding robotiq control

* adding gripper to the URDF and dependency update

* updating launch

* updating ur_control launch

* removing the unwanted RViz node

* updates for fake hardware for gripper

* adding a if condition to disable neobotix hardware components for mock

* adding Epick gripper

* updating control launch

---------

Co-authored-by: Adarsh Karan Kesavadas Prasanth <adarshkaran01@gmail.com>

File: robot_model/mpo_700/mpo_700.urdf.xacro (robot description, xacro)
@@ -5,7 +5,11 @@
   <xacro:arg name="use_imu" default="false"/>
   <xacro:arg name="use_d435" default="false"/>
+  <xacro:arg name="gripper_type" default="2f_140"/>
+  <xacro:arg name="use_fake_hardware" default="false"/>
   <xacro:property name="arm" value="$(arg arm_type)"/>
   <xacro:property name="imu" value="$(arg use_imu)"/>
   <xacro:property name="d435" value="$(arg use_d435)"/>
+  <xacro:property name="gripper" value="$(arg gripper_type)"/>
+  <xacro:property name="use_fake" value="$(arg use_fake_hardware)"/>
   <!-- When there is an arm mounted, the joints of the wheels needs
   to be of fixed type. The reason being, both the drive modules and
@@ -392,4 +396,33 @@
       <origin xyz="0.133 0.0 0.416" rpy="0.0 0.0 -1.5708" />
     </xacro:ur_robot>
+    <!-- add gripper-->
+    <xacro:unless value="${gripper == ''}">
+      <!-- ur_adapter for gripper-->
+      <xacro:if value="${gripper == '2f_140'}">
+        <xacro:include filename="$(find robotiq_description)/urdf/ur_to_robotiq_adapter.urdf.xacro"/>
+        <xacro:ur_to_robotiq
+            prefix=""
+            parent="$(arg tf_prefix)tool0"
+            child="neo_gripper_mount_link"
+            rotation="${pi/2}"
+            />
+        <xacro:include filename="$(find robotiq_description)/urdf/robotiq_2f_140_macro.urdf.xacro"/>
+        <xacro:robotiq_gripper name="robotiq_gripper"
+          prefix=""
+          parent="neo_gripper_mount_link"
+          include_ros2_control="true"
+          use_fake_hardware="${use_fake}">
+            <origin xyz="0 0 0" rpy="0 0 -${pi / 2}"/>
+        </xacro:robotiq_gripper>
+      </xacro:if>
+      <xacro:if value="${gripper == 'epick'}">
+        <xacro:include filename="$(find epick_description)/urdf/epick_single_suction_cup.xacro"/>
+          <xacro:epick_single_suction_cup parent="$(arg tf_prefix)tool0"
+            use_fake_hardware="${use_fake}"
+            origin_xyz="0 0 0"
+            origin_rpy="0 0 -${pi / 2}"
+            />
+      </xacro:if>
+    </xacro:unless>
   </xacro:unless>
 </robot>
