Commit message: Added 2f_140 robotiq gripper support

File: robot_model/mpo_700.urdf.xacro (robot description, xacro)
@@ -18,4 +18,5 @@
   <xacro:arg name="force_abs_paths" default="false"/>
   <xacro:arg name="simulation_controllers" default=""/>
+  <xacro:arg name="gripper_simulation_controllers" default=""/>
   <xacro:arg name="use_mock_hardware" default="false"/>
   <xacro:arg name="mock_sensor_commands" default="false"/>
@@ -134,12 +135,23 @@
             include_ros2_control="true"
             use_mock_hardware="${use_mock}"
+            mock_sensor_commands="${use_mock}"
+            sim_gazebo= "${gz}"
             >
             <origin xyz="0 0 0" rpy="0 0 -${pi / 2}"/>
           </xacro:robotiq_gripper>
+            <!-- <gazebo>
+              <plugin filename="gz_ros2_control-system" name="gz_ros2_control::GazeboSimROS2ControlPlugin">
+                <parameters>$(arg gripper_simulation_controllers)</parameters>
+                <controller_manager_name>gripper_controller_manager</controller_manager_name>
+                <ros>
+                    <namespace>robotiq_gripper</namespace>
+                </ros>
+              </plugin>
+            </gazebo> -->
         </xacro:if>
         <xacro:if value="${gripper == 'epick'}">
           <xacro:include filename="$(find epick_description)/urdf/epick_single_suction_cup.xacro"/>
           <xacro:epick_single_suction_cup parent="$(arg tf_prefix)tool0"
-            use_mock_hardware="${use_mock}"
+            use_fake_hardware="${use_mock}"
             origin_xyz="0 0 0"
             origin_rpy="0 0 -${pi / 2}"

File: robot_model/xacros/mpo_700_body.urdf.xacro (robot description, xacro)
@@ -39,5 +39,5 @@
       <origin rpy="0 0 0" xyz="0 0 0"/>
       <axis xyz="0 0 -1"/>
-      <joint_properties damping="1" friction="1"/>
+      <dynamics damping="1" friction="1"/>
       <parent link="base_link"/>
       <child link="base_footprint"/>

Commit message: Minor formatting fixes and removed unused launch arg

File: robot_model/mpo_700.urdf.xacro (robot description, xacro)
@@ -12,5 +12,5 @@
   <xacro:arg name="scanner_type" default="sick_s300"/>
   <xacro:arg name="use_docking_adapter" default="false"/>
-  <!-- Arm Arguments-->
+  <!-- Manipulator Arguments-->
   <xacro:arg name="arm_type" default=""/>
   <xacro:arg name="arm_parent" default="cabinet_link"/>
@@ -119,36 +119,36 @@
       <xacro:include filename="$(find mp_components)/urdf/arm/elite_arm.urdf.xacro"/>
     </xacro:if>
-      <!-- add gripper-->
-      <xacro:unless value="${gripper == ''}">
-        <!-- ur_adapter for gripper-->
-        <xacro:if value="${gripper == '2f_140' or gripper == '2f_85'}">
-          <xacro:include filename="$(find robotiq_description)/urdf/ur_to_robotiq_adapter.urdf.xacro"/>
-          <xacro:ur_to_robotiq
-            prefix=""
-            parent="$(arg tf_prefix)tool0"
-            child="neo_gripper_mount_link"
-            rotation="${pi/2}"
-            />
-          <xacro:include filename="$(find robotiq_description)/urdf/robotiq_${gripper}_macro.urdf.xacro"/>
-          <xacro:robotiq_gripper name="robotiq_gripper"
-            prefix=""
-            parent="neo_gripper_mount_link"
-            use_mock_hardware="${use_mock}"
-            mock_sensor_commands="${use_mock}"
-            sim_gazebo="${gz}"
-            include_ros2_control="$(arg include_gripper_ros2_control)"
-            >
-            <origin xyz="0 0 0" rpy="0 0 -${pi / 2}"/>
-          </xacro:robotiq_gripper>
-        </xacro:if>
-        <xacro:if value="${gripper == 'epick'}">
-          <xacro:include filename="$(find epick_description)/urdf/epick_single_suction_cup.xacro"/>
-          <xacro:epick_single_suction_cup parent="$(arg tf_prefix)tool0"
-            use_fake_hardware="${use_mock}"
-            origin_xyz="0 0 0"
-            origin_rpy="0 0 -${pi / 2}"
-            />
-        </xacro:if>
-      </xacro:unless>
+    <!-- add gripper-->
+    <xacro:unless value="${gripper == ''}">
+      <!-- ur_adapter for gripper-->
+      <xacro:if value="${gripper == '2f_140' or gripper == '2f_85'}">
+        <xacro:include filename="$(find robotiq_description)/urdf/ur_to_robotiq_adapter.urdf.xacro"/>
+        <xacro:ur_to_robotiq
+          prefix=""
+          parent="$(arg tf_prefix)tool0"
+          child="neo_gripper_mount_link"
+          rotation="${pi/2}"
+          />
+        <xacro:include filename="$(find robotiq_description)/urdf/robotiq_${gripper}_macro.urdf.xacro"/>
+        <xacro:robotiq_gripper name="robotiq_gripper"
+          prefix=""
+          parent="neo_gripper_mount_link"
+          use_mock_hardware="${use_mock}"
+          mock_sensor_commands="${use_mock}"
+          sim_gazebo="${gz}"
+          include_ros2_control="$(arg include_gripper_ros2_control)"
+          >
+          <origin xyz="0 0 0" rpy="0 0 -${pi / 2}"/>
+        </xacro:robotiq_gripper>
+      </xacro:if>
+      <xacro:if value="${gripper == 'epick'}">
+        <xacro:include filename="$(find epick_description)/urdf/epick_single_suction_cup.xacro"/>
+        <xacro:epick_single_suction_cup parent="$(arg tf_prefix)tool0"
+          use_fake_hardware="${use_mock}"
+          origin_xyz="0 0 0"
+          origin_rpy="0 0 -${pi / 2}"
+          />
+      </xacro:if>
+    </xacro:unless>
   </xacro:unless>
   <!-- Simulation -->

Commit message: making laser scanner package option

File: robot_model/mpo_700.urdf.xacro (robot description, xacro)
@@ -12,4 +12,5 @@
   <xacro:arg name="scanner_type" default="sick_s300"/>
   <xacro:arg name="use_docking_adapter" default="false"/>
+  <xacro:arg name="disable_scanners" default="false"/>
   <!-- Manipulator Arguments-->
   <xacro:arg name="arm_type" default=""/>
@@ -28,4 +29,5 @@
   <xacro:property name="d435" value="$(arg use_d435)"/>
   <xacro:property name="scanner" value="$(arg scanner_type)"/>
+  <xacro:property name="disable_scanner" value="$(arg disable_scanners)"/>
   <xacro:property name="scanner_height" value="0"/>
   <xacro:property name="gripper" value="$(arg gripper_type)"/>
@@ -46,25 +48,27 @@
   <xacro:mpo_700_body/>
   <!-- Laser Scanners -->
-  <xacro:if value="${scanner == 'sick_s300'}">
-    <!--https://neobotix-docs.de/hardware/en/platforms/mpo-700/mechanical.html-->
-    <xacro:property name="scanner_height" value="0.223"/>
-    <xacro:include filename="$(find neo_mpo_700-2)/robot_model/xacros/sick_s300_macro.xacro"/>
+  <xacro:if value="${disable_scanner == False}">
+    <xacro:if value="${scanner == 'sick_s300'}">
+      <!--https://neobotix-docs.de/hardware/en/platforms/mpo-700/mechanical.html-->
+      <xacro:property name="scanner_height" value="0.223"/>
+      <xacro:include filename="$(find neo_mpo_700-2)/robot_model/xacros/sick_s300_macro.xacro"/>
+    </xacro:if>
+    <xacro:if value="${scanner == 'sick_microscan3'}">
+      <xacro:property name="scanner_height" value="0.223"/>
+      <xacro:include filename="$(find neo_mpo_700-2)/robot_model/xacros/sick_microscan3_macro.xacro"/>
+    </xacro:if>
+    <xacro:sick_laser_scanner
+      name="lidar_1"
+      parent="base_link"
+      >
+      <origin rpy="3.14 0 0.79" xyz="0.338 0.288 ${scanner_height}"/>
+    </xacro:sick_laser_scanner>
+    <xacro:sick_laser_scanner
+      name="lidar_2"
+      parent="base_link"
+      >
+      <origin rpy="3.14 0 3.93" xyz="-0.338 -0.288 ${scanner_height}"/>
+    </xacro:sick_laser_scanner>
   </xacro:if>
-  <xacro:if value="${scanner == 'sick_microscan3'}">
-    <xacro:property name="scanner_height" value="0.223"/>
-    <xacro:include filename="$(find neo_mpo_700-2)/robot_model/xacros/sick_microscan3_macro.xacro"/>
-  </xacro:if>
-  <xacro:sick_laser_scanner
-    name="lidar_1"
-    parent="base_link"
-    >
-    <origin rpy="3.14 0 0.79" xyz="0.338 0.288 ${scanner_height}"/>
-  </xacro:sick_laser_scanner>
-  <xacro:sick_laser_scanner
-    name="lidar_2"
-    parent="base_link"
-    >
-    <origin rpy="3.14 0 3.93" xyz="-0.338 -0.288 ${scanner_height}"/>
-  </xacro:sick_laser_scanner>
   <!-- Using IMU -->
   <xacro:if value="${imu == True}">

Commit message: Added support for ur arm dc cabinet

File: robot_model/mpo_700.urdf.xacro (robot description, xacro)
@@ -17,4 +17,5 @@
   <xacro:arg name="arm_parent" default="cabinet_link"/>
   <xacro:arg name="gripper_type" default=""/>
+  <xacro:arg name="use_ur_dc" default="false"/>
   <xacro:arg name="force_abs_paths" default="false"/>
   <xacro:arg name="simulation_controllers" default=""/>
@@ -32,4 +33,5 @@
   <xacro:property name="scanner_height" value="0"/>
   <xacro:property name="gripper" value="$(arg gripper_type)"/>
+  <xacro:property name="ur_dc" value="$(arg use_ur_dc)"/>
   <xacro:property name="docking_adapter" value="$(arg use_docking_adapter)"/>
   <xacro:property name="use_mock" value="$(arg use_mock_hardware)"/>
@@ -117,8 +119,17 @@
     <!-- Universal Robotics (UR) Arms-->
     <xacro:if value="${arm == 'ur5' or arm == 'ur10' or arm == 'ur5e' or arm == 'ur10e'}">
+      <!-- Different height for AC arm-->
+      <xacro:if value="${ur_dc == False}">
+        <xacro:property name="arm_height" value="0.416" />
+      </xacro:if>
+      <xacro:if value="${ur_dc == True}">
+        <xacro:property name="arm_height" value="0.307" />
+      </xacro:if>
+      <!-- Include the UR arm -->
       <xacro:include filename="$(find mp_components)/urdf/arm/ur_arm.urdf.xacro"/>
     </xacro:if>
     <!-- Elite Arms-->
     <xacro:if value="${arm == 'ec66' or arm == 'cs66'}">
+      <xacro:property name="arm_height" value="0.376" />
       <xacro:include filename="$(find mp_components)/urdf/arm/elite_arm.urdf.xacro"/>
     </xacro:if>

Commit message: updating the arm height for DC controller box

File: robot_model/mpo_700.urdf.xacro (robot description, xacro)
@@ -124,5 +124,5 @@
       </xacro:if>
       <xacro:if value="${ur_dc == True}">
-        <xacro:property name="arm_height" value="0.307" />
+        <xacro:property name="arm_height" value="0.265" />
       </xacro:if>
       <!-- Include the UR arm -->

Commit message: updating height of UR DC

File: robot_model/mpo_700.urdf.xacro (robot description, xacro)
@@ -124,5 +124,5 @@
       </xacro:if>
       <xacro:if value="${ur_dc == True}">
-        <xacro:property name="arm_height" value="0.265" />
+        <xacro:property name="arm_height" value="0.272" />
       </xacro:if>
       <!-- Include the UR arm -->
