Commit message: updating xacros to adapt odm for both sim and real

File: robot_model/xacros/mpo_700_body.urdf.xacro (robot description, xacro)
@@ -9,4 +9,11 @@
   <xacro:include filename="$(find neo_mpo_700-2)/robot_model/xacros/mpo_700_wheel_macro.xacro"/>
   <xacro:macro name="mpo_700_body">
+    <!-- Required for visualizing the left ODM's outwards during the start -->
+    <xacro:property name="angle_comp" value="1"/>
+    <xacro:property name="disp_comp" value="-1"/>
+    <xacro:if value="${ODM_joint_type == 'fixed'}">
+      <xacro:property name="angle_comp" value="0"/>
+      <xacro:property name="disp_comp" value="1"/>
+    </xacro:if>
     <link name="base_link"/>
     <link name="base_footprint">
@@ -48,5 +55,5 @@
       parent_link="base_footprint"
       caster_joint_type="${ODM_joint_type}"
-      link_origin_rpy="0 0 0"
+      link_origin_rpy="0 0 ${3.14 * angle_comp}"
       >
       <origin rpy="0 0 0" xyz="0.24 0.18 0.22"/>
@@ -64,5 +71,5 @@
       parent_link="base_footprint"
       caster_joint_type="${ODM_joint_type}"
-      link_origin_rpy="0 0 0"
+      link_origin_rpy="0 0 ${3.14 * angle_comp}"
       >
       <origin rpy="0 0 0" xyz="-0.24 0.18 0.22"/>
@@ -82,5 +89,5 @@
       wheel_joint_type="${ODM_joint_type}"
       >
-      <origin rpy="0 0 0" xyz="0.0 0.045 -0.12"/>
+      <origin rpy="0 0 ${3.14 * angle_comp}" xyz="0.0 ${0.045 * disp_comp} -0.12"/>
     </xacro:mpo_700_wheel>
     <xacro:mpo_700_wheel
@@ -96,5 +103,5 @@
       wheel_joint_type="${ODM_joint_type}"
       >
-      <origin rpy="0 0 0" xyz="0.0 0.045 -0.12"/>
+      <origin rpy="0 0 ${3.14 * angle_comp}" xyz="0.0 ${0.045 * disp_comp} -0.12"/>
     </xacro:mpo_700_wheel>
     <xacro:mpo_700_wheel

Commit message: updating the robot model for customization

File: robot_model/xacros/mpo_700_body.urdf.xacro (robot description, xacro)
@@ -57,5 +57,5 @@
       link_origin_rpy="0 0 ${3.14 * angle_comp}"
       >
-      <origin rpy="0 0 0" xyz="0.24 0.18 0.22"/>
+      <origin rpy="0 0 0" xyz="0.25 0.18 0.22"/>
     </xacro:mpo_700_caster_wheel>
     <xacro:mpo_700_caster_wheel
@@ -65,5 +65,5 @@
       link_origin_rpy="0 0 3.14"
       >
-      <origin rpy="0 0 0" xyz="0.24 -0.18 0.22"/>
+      <origin rpy="0 0 0" xyz="0.25 -0.18 0.22"/>
     </xacro:mpo_700_caster_wheel>
     <xacro:mpo_700_caster_wheel
@@ -73,5 +73,5 @@
       link_origin_rpy="0 0 ${3.14 * angle_comp}"
       >
-      <origin rpy="0 0 0" xyz="-0.24 0.18 0.22"/>
+      <origin rpy="0 0 0" xyz="-0.25 0.18 0.22"/>
     </xacro:mpo_700_caster_wheel>
     <xacro:mpo_700_caster_wheel
@@ -81,5 +81,5 @@
       link_origin_rpy="0 0 3.14"
       >
-      <origin rpy="0 0 0" xyz="-0.24 -0.18 0.22"/>
+      <origin rpy="0 0 0" xyz="-0.25 -0.18 0.22"/>
     </xacro:mpo_700_caster_wheel>
     <!-- Wheels -->

Commit message: updating the dae files

File: robot_model/xacros/mpo_700_body.urdf.xacro (robot description, xacro)
@@ -57,5 +57,5 @@
       link_origin_rpy="0 0 ${3.14 * angle_comp}"
       >
-      <origin rpy="0 0 0" xyz="0.25 0.18 0.22"/>
+      <origin rpy="0 0 0" xyz="0.25 0.18 0.232"/>
     </xacro:mpo_700_caster_wheel>
     <xacro:mpo_700_caster_wheel
@@ -65,5 +65,5 @@
       link_origin_rpy="0 0 3.14"
       >
-      <origin rpy="0 0 0" xyz="0.25 -0.18 0.22"/>
+      <origin rpy="0 0 0" xyz="0.25 -0.18 0.232"/>
     </xacro:mpo_700_caster_wheel>
     <xacro:mpo_700_caster_wheel
@@ -73,5 +73,5 @@
       link_origin_rpy="0 0 ${3.14 * angle_comp}"
       >
-      <origin rpy="0 0 0" xyz="-0.25 0.18 0.22"/>
+      <origin rpy="0 0 0" xyz="-0.25 0.18 0.232"/>
     </xacro:mpo_700_caster_wheel>
     <xacro:mpo_700_caster_wheel
@@ -81,5 +81,5 @@
       link_origin_rpy="0 0 3.14"
       >
-      <origin rpy="0 0 0" xyz="-0.25 -0.18 0.22"/>
+      <origin rpy="0 0 0" xyz="-0.25 -0.18 0.232"/>
     </xacro:mpo_700_caster_wheel>
     <!-- Wheels -->
@@ -89,5 +89,5 @@
       wheel_joint_type="${ODM_joint_type}"
       >
-      <origin rpy="0 0 ${3.14 * angle_comp}" xyz="0.0 ${0.045 * disp_comp} -0.12"/>
+      <origin rpy="0 0 ${3.14 * angle_comp}" xyz="0.0 ${0.045 * disp_comp} -0.142"/>
     </xacro:mpo_700_wheel>
     <xacro:mpo_700_wheel
@@ -96,5 +96,5 @@
       wheel_joint_type="${ODM_joint_type}"
       >
-      <origin rpy="0 0 3.14" xyz="0.0 -0.045 -0.12"/>
+      <origin rpy="0 0 3.14" xyz="0.0 -0.045 -0.142"/>
     </xacro:mpo_700_wheel>
     <xacro:mpo_700_wheel
@@ -103,5 +103,5 @@
       wheel_joint_type="${ODM_joint_type}"
       >
-      <origin rpy="0 0 ${3.14 * angle_comp}" xyz="0.0 ${0.045 * disp_comp} -0.12"/>
+      <origin rpy="0 0 ${3.14 * angle_comp}" xyz="0.0 ${0.045 * disp_comp} -0.142"/>
     </xacro:mpo_700_wheel>
     <xacro:mpo_700_wheel
@@ -110,5 +110,5 @@
       wheel_joint_type="${ODM_joint_type}"
       >
-      <origin rpy="0 0 3.14" xyz="0.0 -0.045 -0.12"/>
+      <origin rpy="0 0 3.14" xyz="0.0 -0.045 -0.142"/>
     </xacro:mpo_700_wheel>
   </xacro:macro>
